Commit message: Add grasp reachability sweep functionality and evaluation service
- Updated `grasp_waypoint_test.launch.py` to include parameters for sweep mode and CSV output.
- Introduced `grasp_reachability_sweep.py` script to perform reachability sweeps and log results.
- Added `EvaluateBoxPose.srv` service for evaluating box poses.
- Modified `CMakeLists.txt` and `package.xml` to include dependencies for new service and script.
- Enhanced `DualArmGraspWaypointPlanner.cpp` to integrate the evaluation service and handle dry-run mode.
- Adjusted URDF files for correct joint configurations.

File: src/ocs2_robotic_assets/resources/gensong_board/urdf/gensong_board.urdf (robot description, URDF)
Before this commit: robot gsrobot_description, 29 links, 28 joints
Joints:
- joint wheel_drive_left_joint: axis 0 -1 0 -> 0 1 0
- joint wheel_driven_left_joint: type fixed -> continuous
- joint wheel_driven_right_joint: axis 0 -1 0 -> 0 1 0; type fixed -> continuous
